File: pcb/KiCAD/kv4p-ht-PANEL/kv4p-ht-PANEL.kicad_pcb (KiCad board)
At the start: 4 copper layers, 81.2 x 96.6 mm, 178 parts, among them J1 Antenna, J2 SMA, J4 SAO v.69bis, J5 USB-C Socket, J6 GPIO Header, Q1 SS8050, Q2 SS8050, Q3 AO3400A, SW1 PTT, SW2 PTT, SW3 Reset, SW4 Program, U1 DRA/SA818, U2 AZ1117H-3.3TRG1, U4 CP2102N-A02-GQFN24, U5 ESP32-WROOM-32E-N4

Commit message: v2.0d. #175 Larger 818 pads. Removed unused outlines. ADC Biasing.
Parts:
- removed the C10 at (133.3, 61.9)
- removed the C10 at (176.4, 61.9)
- removed the C11 at (127.0, 64.5)
- removed the C11 at (170.1, 64.5)
- removed the C12 at (131.4, 61.9)
- removed the C12 at (174.5, 61.9)
- removed the C13 at (166.9, 61.9)
- removed the C13 at (123.8, 61.9)
- removed the C14 at (187.6, 36.5)
- removed the C14 at (144.5, 36.5)
- removed the C2 at (118.1, 61.9)
- removed the C2 at (161.2, 61.9)
- removed the C3 at (110.4, 59.4)
- removed the C3 at (153.5, 59.4)
- removed the C7 at (115.5, 61.3)
- removed the C7 at (158.6, 61.3)
- removed the C8 at (157.0, 36.5)
- removed the C8 at (113.9, 36.5)
- removed D2 (x2): Red, LED_SMD:LED_0603_1608Metric
- removed the D3 at (174.5, 67.6)
- removed the D3 at (131.4, 67.6)
- removed the D4 at (165.6, 67.6)
- removed the D4 at (122.5, 67.6)
- removed the G*** at (170.1, 50.5)
- removed the G*** at (127.0, 50.5)
- removed J2 (x2): SMA, Connector_Coaxial:SMA_Molex_73251-2120_EdgeMount_Horizontal
- removed the Q3 at (159.9, 66.4)
- removed the Q3 at (116.8, 66.4)
- removed the R15 at (174.5, 66.4)
- removed the R15 at (131.4, 66.4)
- removed R17 (x2): 0R, Resistor_SMD:R_0603_1608Metric
- removed the R2 at (139.7, 37.8)
- removed the R2 at (182.8, 37.8)
- removed the R20 at (122.5, 66.4)
- removed the R20 at (165.6, 66.4)
- removed R22 (x2): 47k, Resistor_SMD:R_0603_1608Metric
- removed the R3 at (142.2, 37.8)
- removed the R3 at (185.3, 37.8)
- removed the R4 at (165.6, 61.9)
- removed the R4 at (122.5, 61.9)
- removed the R5 at (173.2, 61.9)
- removed the R5 at (130.1, 61.9)
- removed the SW3 at (122.5, 71.5)
- removed the SW3 at (165.6, 71.5)
- removed the SW4 at (174.5, 71.5)
- removed the SW4 at (131.4, 71.5)
- removed the TP3 at (187.2, 102.6)
- removed the TP3 at (144.1, 102.6)
- removed the TP4 at (184.7, 36.0)
- removed the TP4 at (141.6, 36.0)
- removed the TP5 at (176.4, 59.8)
- removed the TP5 at (133.3, 59.8)
- removed the U1 at (127.6, 48.6)
- removed the U1 at (170.7, 48.6)
- added C10: 1uF, Capacitor_SMD:C_0603_1608Metric, F.Cu at (133.3, 62.2)
- added C10: 1uF, Capacitor_SMD:C_0603_1608Metric, F.Cu at (176.4, 62.2)
- added C11: 100nF, Capacitor_SMD:C_0603_1608Metric, F.Cu at (127.0, 63.8)
- added C11: 100nF, Capacitor_SMD:C_0603_1608Metric, F.Cu at (170.1, 63.8)
- added C12: 2.2nF Tuned VHF, Capacitor_SMD:C_0603_1608Metric, F.Cu at (131.4, 62.2)
- added C12: 2.2nF Tuned VHF, Capacitor_SMD:C_0603_1608Metric, F.Cu at (174.5, 62.2)
- added C13: 2.2nF Tuned VHF, Capacitor_SMD:C_0603_1608Metric, F.Cu at (166.9, 62.2)
- added C13: 2.2nF Tuned VHF, Capacitor_SMD:C_0603_1608Metric, F.Cu at (123.8, 62.2)
- added C14: 2.2nF Tuned VHF, Capacitor_SMD:C_0603_1608Metric, F.Cu at (144.2, 36.8)
- added C14: 2.2nF Tuned VHF, Capacitor_SMD:C_0603_1608Metric, F.Cu at (187.3, 36.8)
- added C2: 100uF 6.3v, Capacitor_Tantalum_SMD:CP_EIA-3528-21_Kemet-B, F.Cu at (117.6, 62.7)
- added C2: 100uF 6.3v, Capacitor_Tantalum_SMD:CP_EIA-3528-21_Kemet-B, F.Cu at (160.7, 62.7)
- added C23: 2.2nF Tuned VHF, Capacitor_SMD:C_0603_1608Metric, F.Cu at (177.7, 62.2)
- added C23: 2.2nF Tuned VHF, Capacitor_SMD:C_0603_1608Metric, F.Cu at (134.6, 62.2)
- added C24: 2.2nF Tuned VHF, Capacitor_SMD:C_0603_1608Metric, F.Cu at (184.8, 33.2)
- added C24: 2.2nF Tuned VHF, Capacitor_SMD:C_0603_1608Metric, F.Cu at (141.7, 33.2)
- added C3: 2.2nF Tuned VHF, Capacitor_SMD:C_0603_1608Metric, F.Cu at (153.5, 58.9)
- added C3: 2.2nF Tuned VHF, Capacitor_SMD:C_0603_1608Metric, F.Cu at (110.4, 58.9)
- added C7: 100nF, Capacitor_SMD:C_0603_1608Metric, F.Cu at (158.2, 61.9)
- added C7: 100nF, Capacitor_SMD:C_0603_1608Metric, F.Cu at (115.1, 61.9)
- added C8: 2.2nF Tuned VHF, Capacitor_SMD:C_0603_1608Metric, F.Cu at (157.0, 36.1)
- added C8: 2.2nF Tuned VHF, Capacitor_SMD:C_0603_1608Metric, F.Cu at (113.9, 36.1)
- added D3: Red, LED_SMD:LED_0603_1608Metric, F.Cu at (174.4, 65.2)
- added D3: Red, LED_SMD:LED_0603_1608Metric, F.Cu at (131.3, 65.2)
- added D4: Red, LED_SMD:LED_0603_1608Metric, F.Cu at (165.7, 65.2)
- added D4: Red, LED_SMD:LED_0603_1608Metric, F.Cu at (122.6, 65.2)
- added G***: LOGO, kv4p-ht:qr-code, B.Cu at (172.6, 51.9)
- added G***: LOGO, kv4p-ht:qr-code, B.Cu at (129.5, 51.9)
- added Q3: AO3400A, Package_TO_SOT_SMD:SOT-23, F.Cu at (159.9, 66.9)
- added Q3: AO3400A, Package_TO_SOT_SMD:SOT-23, F.Cu at (116.8, 66.9)
- added R15: 1.2k, Resistor_SMD:R_0603_1608Metric, F.Cu at (128.7, 65.4)
- added R15: 1.2k, Resistor_SMD:R_0603_1608Metric, F.Cu at (171.8, 65.4)
- added R2: 10k, Resistor_SMD:R_0603_1608Metric, F.Cu at (139.1, 36.8)
- added R2: 10k, Resistor_SMD:R_0603_1608Metric, F.Cu at (182.2, 36.8)
- added R20: 10k, Resistor_SMD:R_0603_1608Metric, F.Cu at (125.2, 65.4)
- added R20: 10k, Resistor_SMD:R_0603_1608Metric, F.Cu at (168.3, 65.4)
- added R3: 1.2k, Resistor_SMD:R_0603_1608Metric, F.Cu at (141.7, 36.8)
- added R3: 1.2k, Resistor_SMD:R_0603_1608Metric, F.Cu at (184.8, 36.8)
- added R4: 100R, Resistor_SMD:R_0603_1608Metric, F.Cu at (165.6, 62.2)
- added R4: 100R, Resistor_SMD:R_0603_1608Metric, F.Cu at (122.5, 62.2)
- added R5: 100R, Resistor_SMD:R_0603_1608Metric, F.Cu at (173.2, 62.2)
- added R5: 100R, Resistor_SMD:R_0603_1608Metric, F.Cu at (130.1, 62.2)
- added SW3: Reset, Button_Switch_SMD:SW_SPST_TL3342, F.Cu at (121.5, 70.2)
- added SW3: Reset, Button_Switch_SMD:SW_SPST_TL3342, F.Cu at (164.6, 70.2)
- added SW4: Program, Button_Switch_SMD:SW_SPST_TL3342, F.Cu at (175.5, 70.2)
- added SW4: Program, Button_Switch_SMD:SW_SPST_TL3342, F.Cu at (132.4, 70.2)
- added TP3: Gnd, TestPoint:TestPoint_THTPad_D2.5mm_Drill1.2mm, F.Cu at (144.1, 102.6)
- added TP3: Gnd, TestPoint:TestPoint_THTPad_D2.5mm_Drill1.2mm, F.Cu at (187.2, 102.6)
- added TP4: Radio Mic, TestPoint:TestPoint_Pad_D1.5mm, F.Cu at (141.6, 35.3)
- added TP4: Radio Mic, TestPoint:TestPoint_Pad_D1.5mm, F.Cu at (184.7, 35.3)
- added TP5: Radio AF Out, TestPoint:TestPoint_Pad_D1.5mm, F.Cu at (178.9, 61.4)
- added TP5: Radio AF Out, TestPoint:TestPoint_Pad_D1.5mm, F.Cu at (135.8, 61.4)
- added U1: DRA/SA818, kv4p-ht:DORJI_DRA818V, F.Cu at (127.6, 48.6)
- added U1: DRA/SA818, kv4p-ht:DORJI_DRA818V, F.Cu at (170.7, 48.6)
Connections:
- net Board_0-/SAO GPIO1 renamed Board_0-/GPIO27
- net Board_1-/SAO GPIO1 renamed Board_1-/GPIO27
- J4 pad 5: Board_0-/SAO GPIO0 -> Board_0-/GPIO32
- J4 pad 5: Board_1-/SAO GPIO0 -> Board_1-/GPIO32
- R1 pad 1: Board_0-GND -> Board_0-/ADC Bias
- R1 pad 1: Board_1-GND -> Board_1-/ADC Bias
- U5 pad 11: Board_0-/SAO GPIO0 -> Board_0-/ADC Bias
- U5 pad 5: Board_0-+3.3V -> Board_0-GND
- U5 pad 11: Board_1-/SAO GPIO0 -> Board_1-/ADC Bias
- U5 pad 5: Board_1-+3.3V -> Board_1-GND
Routing:
- net Board_1-/SAO GPIO0: track 14.3 -> 0.00 mm, vias 2 -> 0
- net Board_0-/SAO GPIO0: track 14.3 -> 0.00 mm, vias 2 -> 0
- net Board_0-/ADC Bias: track 0.00 -> 8.12 mm, vias 0 -> 2
- net Board_1-/ADC Bias: track 0.00 -> 8.12 mm, vias 0 -> 2
- net Board_1-+3.3V: track 92.4 -> 97.3 mm, vias 7 -> 9
- net Board_0-+3.3V: track 92.4 -> 97.3 mm, vias 7 -> 9
- net Board_1-/Stock LED: track 16.3 -> 19.8 mm
- net Board_0-/Stock LED: track 16.3 -> 19.8 mm
- net Board_0-+5V: track 38.7 -> 35.6 mm, vias 162 -> 152
- net Board_1-+5V: track 38.7 -> 35.6 mm, vias 162 -> 152
- net Board_1-Net-(J1-In): track 12.1 -> 9.06 mm
- net Board_0-Net-(J1-In): track 12.1 -> 9.06 mm
- net Board_1-/Radio Mic In: track 4.28 -> 7.20 mm
- net Board_0-/Radio Mic In: track 4.28 -> 7.20 mm
- net Board_1-/NeoPixel DO: track 22.7 -> 19.9 mm
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Other:
- board text added: "GND"
- board text added: "High Low"
- board text added: "Manufactured by Halibut Electronics, 2025-01-15"
- board text added: "Mic"
- board text added: "Pwr LED"
- board text added: "RF Out"
- board text added: "Ser Rx"
- board text added: "Ser Tx"
- board text added: "Spkr"
- board text added: "Squelch"
- board text added: "User LED"
- board text added: "kv4p HT, v2.0d 2025-01-15 VanceVagell v2 hardware by @SmittyHalibut"
- board text added: "kv4p-ht, v2.0d"
- board text added: "~{PD}"
- board text added: "~{PTT}"
- board text removed: "IO26"
- board text removed: "Manufactured by Halibut Electronics, 2024-12-09"
- board text removed: "Pwr"
- board text removed: "User"
- board text removed: "kv4p HT, v2.0c 2024-12-09 VanceVagell v2 hardware by @SmittyHalibut"
- board text removed: "kv4p-ht, v2.0c"
